File: HW2/PIC32_board/HW2_ME433.brd (EAGLE design)
At the start: 160 x 100 mm, 23 parts, among them J1 USB-MB-H

Commit message: Add files via upload
Parts:
- U$1: device HW2_ME433:QFN44ML8X8 -> HW2_ME433:TQFP44
